File: hardware/expansion-board-v3.1/kicad/rf1090.kicad_sch (KiCad schematic)
At the start: 49 parts, among them J6 U.FL_1090_EXT(经尾线转SMA), Q3 AO3401A, U11 QPL9547TR7, U12 BGA2817, U13 AD8319ACPZ-R7(主), U14 AD8313ARMZ(备,二选一), U15 TLV3501(TOKMAS), U16 XA17-G4K(或AS179-92LF)

Commit message: chore(hw): 工程改名 v1→v3.1、清掉过程文件；板子跑回 plain 流程（未连通 16 / DRC 0）
## 改名

文件名一直叫 expansion-board-v1，而工程早就是 v3.1（六层板），看着容易搞错版本。
统一改成 expansion-board-v3.1：

  kicad/expansion-board-v3.1.{kicad_pcb,kicad_pro,kicad_sch,kicad_sym}
  kicad/expansion-board-v3.1.pretty/          （7 个自制封装）
  kicad/expansion-board-v3.1-{erc.rpt,schematic-REVIEW.pdf}

连带改掉 34 个文件里的 242 处引用（tools/*.py 22 个、两个 .sh、fp/sym-lib-table、
6 张子原理图里的库前缀）。⚠️ 子原理图里的引用最多（rf1090 60 处、sensors 45 处、
subghz 33 处、mcu 31 处），是符号库前缀 expansion-board-v1:XXX，漏改会导致
原理图打开后满屏问号。.kicad_pcb 里 0 处——它的 footprint 不带库前缀。

改完自检：PCB 加载 156 元件 / 封装 ID 缺失 0，网表导出 152 元件，gen_pcb 重建通过。

## 清掉的过程文件

  ~expansion-board-v1.kicad_pcb.lck / .kicad_pro.lck   8/4 的陈旧锁，KiCad 崩溃残留
  Archive.zip (274KB)                                  KiCad 归档，未跟踪
  expansion-board-v1.kicad_prl                         KiCad 本地视图状态

后两类顺手加进 .gitignore（kicad/*.kicad_prl、build/trial/），免得再混进暂存区
——这次 git add -A 就把试验副本 build/trial 和重新生成的 .kicad_prl 卷进来了。
erc.rpt 和 schematic-REVIEW.pdf 保留（评审记录），只跟着改名。

## 板子跑回 plain 流程

上一版 af73179 是 keepout 流程的产物（17 未连通），实测不如 plain。这次用改好
bug 的工具重跑一遍 plain（reroute.sh 那条路），没动 git 历史：

              af73179(keepout)   本次(plain)
  未连通            17              **16**
  铜层 DRC           0                0
  射频            116 段(自布)      156 段(freerouting)

check_route 四条硬约束全过：In1 参考面完整 / 射频 156 段全在 F.Cu / 射频 0 过孔。
剩 12 处真缺线（6 条 RF + 6 条数字），与 e917f2a 同一水平。
Parts:
- ANT1: footprint expansion-board-v1:ANT_IFA_1090MHz -> expansion-board-v3.1:ANT_IFA_1090MHz
- FL1, FL2: footprint expansion-board-v1:TA0970A_SMD3838-6 -> expansion-board-v3.1:TA0970A_SMD3838-6; symbol expansion-board-v1:TA0970A -> expansion-board-v3.1:TA0970A
- U13: footprint expansion-board-v1:AD8319_LFCSP-8-EP -> expansion-board-v3.1:AD8319_LFCSP-8-EP; symbol expansion-board-v1:AD8319 -> expansion-board-v3.1:AD8319
