File: hardware/expansion-board-v3.1/kicad/sensors.kicad_sch (KiCad schematic)
At the start: 30 parts, among them J2 U.FL_GNSS_EXT(经尾线转SMA), J8 U.FL→内置patch, Q4 AO3401A, Q5 AO3401A, U17 XA17-G4K(或AS179-92LF), U4 BNO085, U5 BMP388, U6 QMC5883P, U7 ATGM336H-6N-74

Commit message: chore(hw): 工程改名 v1→v3.1、清掉过程文件；板子跑回 plain 流程（未连通 16 / DRC 0）
## 改名

文件名一直叫 expansion-board-v1，而工程早就是 v3.1（六层板），看着容易搞错版本。
统一改成 expansion-board-v3.1：

  kicad/expansion-board-v3.1.{kicad_pcb,kicad_pro,kicad_sch,kicad_sym}
  kicad/expansion-board-v3.1.pretty/          （7 个自制封装）
  kicad/expansion-board-v3.1-{erc.rpt,schematic-REVIEW.pdf}

连带改掉 34 个文件里的 242 处引用（tools/*.py 22 个、两个 .sh、fp/sym-lib-table、
6 张子原理图里的库前缀）。⚠️ 子原理图里的引用最多（rf1090 60 处、sensors 45 处、
subghz 33 处、mcu 31 处），是符号库前缀 expansion-board-v1:XXX，漏改会导致
原理图打开后满屏问号。.kicad_pcb 里 0 处——它的 footprint 不带库前缀。

改完自检：PCB 加载 156 元件 / 封装 ID 缺失 0，网表导出 152 元件，gen_pcb 重建通过。

## 清掉的过程文件

  ~expansion-board-v1.kicad_pcb.lck / .kicad_pro.lck   8/4 的陈旧锁，KiCad 崩溃残留
  Archive.zip (274KB)                                  KiCad 归档，未跟踪
  expansion-board-v1.kicad_prl                         KiCad 本地视图状态

后两类顺手加进 .gitignore（kicad/*.kicad_prl、build/trial/），免得再混进暂存区
——这次 git add -A 就把试验副本 build/trial 和重新生成的 .kicad_prl 卷进来了。
erc.rpt 和 schematic-REVIEW.pdf 保留（评审记录），只跟着改名。

## 板子跑回 plain 流程

上一版 af73179 是 keepout 流程的产物（17 未连通），实测不如 plain。这次用改好
bug 的工具重跑一遍 plain（reroute.sh 那条路），没动 git 历史：

              af73179(keepout)   本次(plain)
  未连通            17              **16**
  铜层 DRC           0                0
  射频            116 段(自布)      156 段(freerouting)

check_route 四条硬约束全过：In1 参考面完整 / 射频 156 段全在 F.Cu / 射频 0 过孔。
剩 12 处真缺线（6 条 RF + 6 条数字），与 e917f2a 同一水平。
Parts:
- U4: footprint expansion-board-v1:BNO085_LGA-28 -> expansion-board-v3.1:BNO085_LGA-28; symbol expansion-board-v1:BNO085 -> expansion-board-v3.1:BNO085
- U5: footprint expansion-board-v1:BMP388_LGA-10 -> expansion-board-v3.1:BMP388_LGA-10; symbol expansion-board-v1:BMP388 -> expansion-board-v3.1:BMP388
- U6: symbol expansion-board-v1:QMC5883P -> expansion-board-v3.1:QMC5883P
- U7: footprint expansion-board-v1:ATGM336H_LCC-18 -> expansion-board-v3.1:ATGM336H_LCC-18; symbol expansion-board-v1:ATGM336H -> expansion-board-v3.1:ATGM336H
Changed lines of the file:
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@@
 	)
 	(symbol
-		(lib_id "expansion-board-v1:BNO085")
+		(lib_id "expansion-board-v3.1:BNO085")
 		(at 76.2 76.2 0)
 		(unit 1)
@@
 			(effects (font (size 1.27 1.27)))
 		)
-		(property "Footprint" "expansion-board-v1:BNO085_LGA-28"
+		(property "Footprint" "expansion-board-v3.1:BNO085_LGA-28"
 			(at 76.2 81.28 0)
 			(effects (font (size 1.27 1.27))
@@
 		)
 		(instances
-			(project "expansion-board-v1"
+			(project "expansion-board-v3.1"
 				(path "/10000000-0000-4000-8000-000000000001/20000000-0000-4000-8000-000000000005"
 					(reference "U4")
@@
 		)
 		(instances
-			(project "expansion-board-v1"
+			(project "expansion-board-v3.1"
 				(path "/10000000-0000-4000-8000-000000000001/20000000-0000-4000-8000-000000000005"
 					(reference "C10")
@@
 		)
 		(instances
-			(project "expansion-board-v1"
+			(project "expansion-board-v3.1"
 				(path "/10000000-0000-4000-8000-000000000001/20000000-0000-4000-8000-000000000005"
 					(reference "C11")
@@
 		)
 		(instances
-			(project "expansion-board-v1"
+			(project "expansion-board-v3.1"
 				(path "/10000000-0000-4000-8000-000000000001/20000000-0000-4000-8000-000000000005"
 					(reference "C12")
@@
 		)
 		(instances
-			(project "expansion-board-v1"
+			(project "expansion-board-v3.1"
 				(path "/10000000-0000-4000-8000-000000000001/20000000-0000-4000-8000-000000000005"
 					(reference "R1")
@@
 		)
 		(instances
-			(project "expansion-board-v1"
+			(project "expansion-board-v3.1"
 				(path "/10000000-0000-4000-8000-000000000001/20000000-0000-4000-8000-000000000005"
 					(reference "R2")
@@
 		)
 		(instances
-			(project "expansion-board-v1"
+			(project "expansion-board-v3.1"
 				(path "/10000000-0000-4000-8000-000000000001/20000000-0000-4000-8000-000000000005"
 					(reference "R3")
@@
 	)
 	(symbol
-		(lib_id "expansion-board-v1:BMP388")
+		(lib_id "expansion-board-v3.1:BMP388")
 		(at 76.2 137.16 0)
 		(unit 1)
@@
 			(effects (font (size 1.27 1.27)))
 		)
-		(property "Footprint" "expansion-board-v1:BMP388_LGA-10"
+		(property "Footprint" "expansion-board-v3.1:BMP388_LGA-10"
 			(at 76.2 142.24 0)
 			(effects (font (size 1.27 1.27))
@@
 		)
 		(instances
-			(project "expansion-board-v1"
+			(project "expansion-board-v3.1"
 				(path "/10000000-0000-4000-8000-000000000001/20000000-0000-4000-8000-000000000005"
 					(reference "U5")
@@
 		)
 		(instances
-			(project "expansion-board-v1"
+			(project "expansion-board-v3.1"
 				(path "/10000000-0000-4000-8000-000000000001/20000000-0000-4000-8000-000000000005"
 					(reference "C13")
@@
 		)
 		(instances
-			(project "expansion-board-v1"
+			(project "expansion-board-v3.1"
 				(path "/10000000-0000-4000-8000-000000000001/20000000-0000-4000-8000-000000000005"
 					(reference "C14")
@@
 	)
 	(symbol
-		(lib_id "expansion-board-v1:QMC5883P")
+		(lib_id "expansion-board-v3.1:QMC5883P")
 		(at 76.2 185.42 0)
 		(unit 1)
@@
 		)
 		(instances
-			(project "expansion-board-v1"
+			(project "expansion-board-v3.1"
 				(path "/10000000-0000-4000-8000-000000000001/20000000-0000-4000-8000-000000000005"
 					(reference "U6")
@@
 		)
 		(instances
-			(project "expansion-board-v1"
+			(project "expansion-board-v3.1"
 				(path "/10000000-0000-4000-8000-000000000001/20000000-0000-4000-8000-000000000005"
 					(reference "C15")
@@
 		)
 		(instances
-			(project "expansion-board-v1"
+			(project "expansion-board-v3.1"
 				(path "/10000000-0000-4000-8000-000000000001/20000000-0000-4000-8000-000000000005"
 					(reference "C16")
@@
 	)
 	(symbol
-		(lib_id "expansion-board-v1:ATGM336H")
+		(lib_id "expansion-board-v3.1:ATGM336H")
 		(at 190.5 137.16 0)
 		(unit 1)
@@
 			(effects (font (size 1.27 1.27)))
 		)
-		(property "Footprint" "expansion-board-v1:ATGM336H_LCC-18"
+		(property "Footprint" "expansion-board-v3.1:ATGM336H_LCC-18"
 			(at 190.5 142.24 0)
 			(effects (font (size 1.27 1.27))
@@
 		)
 		(instances
-			(project "expansion-board-v1"
+			(project "expansion-board-v3.1"
 				(path "/10000000-0000-4000-8000-000000000001/20000000-0000-4000-8000-000000000005"
 					(reference "U7")
@@
 		)
 		(instances
-			(project "expansion-board-v1"
+			(project "expansion-board-v3.1"
 				(path "/10000000-0000-4000-8000-000000000001/20000000-0000-4000-8000-000000000005"
 					(reference "C57")
@@
 		)
 		(instances
-			(project "expansion-board-v1"
+			(project "expansion-board-v3.1"
 				(path "/10000000-0000-4000-8000-000000000001/20000000-0000-4000-8000-000000000005"
 					(reference "U17")
@@
 		)
 		(instances
-			(project "expansion-board-v1"
+			(project "expansion-board-v3.1"
 				(path "/10000000-0000-4000-8000-000000000001/20000000-0000-4000-8000-000000000005"
 					(reference "C58")
@@
 		)
 		(instances
-			(project "expansion-board-v1"
+			(project "expansion-board-v3.1"
 				(path "/10000000-0000-4000-8000-000000000001/20000000-0000-4000-8000-000000000005"
 					(reference "Q4")
@@
 		)
 		(instances
-			(project "expansion-board-v1"
+			(project "expansion-board-v3.1"
 				(path "/10000000-0000-4000-8000-000000000001/20000000-0000-4000-8000-000000000005"
 					(reference "F4")
@@
 		)
 		(instances
-			(project "expansion-board-v1"
+			(project "expansion-board-v3.1"
 				(path "/10000000-0000-4000-8000-000000000001/20000000-0000-4000-8000-000000000005"
 					(reference "L2")
@@
 		)
 		(instances
-			(project "expansion-board-v1"
+			(project "expansion-board-v3.1"
 				(path "/10000000-0000-4000-8000-000000000001/20000000-0000-4000-8000-000000000005"
 					(reference "C59")
@@
 		)
 		(instances
-			(project "expansion-board-v1"
+			(project "expansion-board-v3.1"
 				(path "/10000000-0000-4000-8000-000000000001/20000000-0000-4000-8000-000000000005"
 					(reference "Q5")
@@
 		)
 		(instances
-			(project "expansion-board-v1"
+			(project "expansion-board-v3.1"
 				(path "/10000000-0000-4000-8000-000000000001/20000000-0000-4000-8000-000000000005"
 					(reference "F5")
@@
 		)
 		(instances
-			(project "expansion-board-v1"
+			(project "expansion-board-v3.1"
 				(path "/10000000-0000-4000-8000-000000000001/20000000-0000-4000-8000-000000000005"
 					(reference "L15")
@@
 		)
 		(instances
-			(project "expansion-board-v1"
+			(project "expansion-board-v3.1"
 				(path "/10000000-0000-4000-8000-000000000001/20000000-0000-4000-8000-000000000005"
 					(reference "J8")
@@
 		)
 		(instances
-			(project "expansion-board-v1"
+			(project "expansion-board-v3.1"
 				(path "/10000000-0000-4000-8000-000000000001/20000000-0000-4000-8000-000000000005"
 					(reference "R26")
@@
 		)
 		(instances
-			(project "expansion-board-v1"
+			(project "expansion-board-v3.1"
 				(path "/10000000-0000-4000-8000-000000000001/20000000-0000-4000-8000-000000000005"
 					(reference "R27")
@@
 		)
 		(instances
-			(project "expansion-board-v1"
+			(project "expansion-board-v3.1"
 				(path "/10000000-0000-4000-8000-000000000001/20000000-0000-4000-8000-000000000005"
 					(reference "C17")
@@
 		)
 		(instances
-			(project "expansion-board-v1"
+			(project "expansion-board-v3.1"
 				(path "/10000000-0000-4000-8000-000000000001/20000000-0000-4000-8000-000000000005"
 					(reference "C18")
@@
 		)
 		(instances
-			(project "expansion-board-v1"
+			(project "expansion-board-v3.1"
 				(path "/10000000-0000-4000-8000-000000000001/20000000-0000-4000-8000-000000000005"
 					(reference "J2")
