File: hardware/expansion-board-v3/kicad/subghz.kicad_sch (KiCad schematic)
At the start: 32 parts, among them J5 U.FL_978, Q2 AO3401A, U10 CC1312R1F3RGZR, Y2 48MHz ABM8W-7pF, Y3 32.768kHz FC-135

Commit message: feat(v3): backport V4 fixes into a clean V3.9 candidate (phases A-D)
Builds the V3.9 candidate from the V3.8 master rather than from the
working-tree intermediate. The intermediate had the 14 audit parts and a
cleared back side, but had lost 24 board-level silkscreen strings and all
four named RF zones - tools/rebuild.sh starts with gen_pcb.py, which calls
pcbnew.NewBoard(), and neither gr_text nor named zones live in
PLACEMENT.py or ROUTES.json, so every run drops them. The master is the
opposite: intact silkscreen and zones, missing only components. Adding
components back is enumerable (14 designators); restoring 24 silkscreen
strings with correct position, layer, size and mirroring is not.

Coordinates are transplanted from the intermediate, so nothing is
re-placed by hand. What that does cost is copper: the master was routed
without these parts, and 13 of the 18 land on existing tracks. Ripping
those out plus the resulting dangling chains removes 176 segments and 26
vias against the master's 1620/377 - all of it folded into phase E, which
was going to be manual routing anyway. Re-placing 13 parts on a fully
routed board would have been worse; C82-C86 are RP2040 local decouplers
that must stay next to the die, which is exactly how V4.3 ended up with
its 30 mm detour.

Phase B removes the AD8319 experimental branch (U13, R20, DET_TADJ). The
"directional error" turned out to reach into the generators, not just
prose - five places, of which two would have produced wrong hardware:

    gen_bom_smt.py   SKIP_REF = {"U14"}   the only detector excluded
                                          from the pick-and-place BOM
    gen_bom.py       ORDERED listed "AD8313ARMZ(备,二选一)", a suffixed
                     string that never matched the netlist value, so the
                     part had never once been classified

Ordering the V3.8 BOM as it stood would have produced a board whose 1090
receive chain has no detector at all. Phase B's hard criterion now holds:
excluding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
Parts:
- added R47, R56: 10k, Resistor_SMD:R_0603_1608Metric, symbol Device:R
- C68: value 12pF -> 18pF
- C69: value 15pF -> 18pF
- D3: value ESD 3.3V/0.6pF -> TPESD8L3.3 0.3pFtyp 0.5pFmax
Connections:
- net 3V3_DIG: now also R17.1, R47.1, R56.1
- net 3V3_GNSS: no longer R17.1
- net SUBG_CSN: now also R56.2
- net SUBG_RESET: now also R47.2
Changed lines of the file:
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@@
+	)
+	(symbol
+		(lib_id "Device:R")
+		(at 127 114.3 0)
+		(unit 1)
+		(exclude_from_sim no)
+		(in_bom yes)
+		(on_board yes)
+		(dnp no)
+		(property "Reference" "R47"
+			(at 127 111.76 0)
+			(effects (font (size 1.27 1.27)))
+		)
+		(property "Value" "10k"
+			(at 127 116.84 0)
+			(effects (font (size 1.27 1.27)))
+		)
+		(property "Footprint" "Resistor_SMD:R_0603_1608Metric"
+			(at 127 119.38 0)
+			(effects (font (size 1.27 1.27))
+				(hide yes))
+		)
+		(property "Datasheet" "~"
+			(at 127 121.92 0)
+			(effects (font (size 1.27 1.27))
+				(hide yes))
+		)
+		(pin "1"
+		)
+		(pin "2"
+		)
+		(instances
+			(project "expansion-board-v3"
+				(path "/10000000-0000-4000-8000-000000000001/20000000-0000-4000-8000-000000000004"
+					(reference "R47")
+					(unit 1)
+				)
+			)
+		)
+	)
+	(global_label "3V3_DIG"
+		(shape passive)
+		(at 127 110.49 270)
+		(effects (font (size 1.27 1.27)) (justify left))
+	)
+	(global_label "SUBG_RESET"
+		(shape passive)
+		(at 127 118.11 90)
+		(effects (font (size 1.27 1.27)) (justify right))
 	)
 	(symbol
@@
 	(symbol
 		(lib_id "Device:R")
+		(at 228.6 127 0)
+		(unit 1)
+		(exclude_from_sim no)
+		(in_bom yes)
+		(on_board yes)
+		(dnp no)
+		(property "Reference" "R56"
+			(at 228.6 124.46 0)
+			(effects (font (size 1.27 1.27)))
+		)
+		(property "Value" "10k"
+			(at 228.6 129.54 0)
+			(effects (font (size 1.27 1.27)))
+		)
+		(property "Footprint" "Resistor_SMD:R_0603_1608Metric"
+			(at 228.6 132.08 0)
+			(effects (font (size 1.27 1.27))
+				(hide yes))
+		)
+		(property "Datasheet" "~"
+			(at 228.6 134.62 0)
+			(effects (font (size 1.27 1.27))
+				(hide yes))
+		)
+		(pin "1"
+		)
+		(pin "2"
+		)
+		(instances
+			(project "expansion-board-v3"
+				(path "/10000000-0000-4000-8000-000000000001/20000000-0000-4000-8000-000000000004"
+					(reference "R56")
+					(unit 1)
+				)
+			)
+		)
+	)
+	(global_label "3V3_DIG"
+		(shape passive)
+		(at 228.6 123.19 270)
+		(effects (font (size 1.27 1.27)) (justify left))
+	)
+	(global_label "SUBG_CSN"
+		(shape passive)
+		(at 228.6 130.81 90)
+		(effects (font (size 1.27 1.27)) (justify right))
+	)
+	(symbol
+		(lib_id "Device:R")
 		(at 190.5 101.6 0)
 		(unit 1)
@@
 		)
 	)
-	(global_label "3V3_GNSS"
+	(global_label "3V3_DIG"
 		(shape passive)
 		(at 190.5 97.79 270)
@@
 			(effects (font (size 1.27 1.27)))
 		)
-		(property "Value" "ESD 3.3V/0.6pF"
+		(property "Value" "TPESD8L3.3 0.3pFtyp 0.5pFmax"
 			(at 254 116.84 0)
 			(effects (font (size 1.27 1.27)))
@@
 			(effects (font (size 1.27 1.27)))
 		)
-		(property "Value" "12pF"
+		(property "Value" "18pF"
 			(at 203.2 154.94 0)
 			(effects (font (size 1.27 1.27)))
@@
 			(effects (font (size 1.27 1.27)))
 		)
-		(property "Value" "15pF"
+		(property "Value" "18pF"
 			(at 215.9 154.94 0)
 			(effects (font (size 1.27 1.27)))
