File: hardware/expansion-board-v4/kicad/expansion-board-v4.kicad_sch (KiCad schematic)
At the start: 0 parts

Commit message: hardware(v4.6): airband BK4819 schematic + symbols + J3 wiring + BOM
- new RF_VHF sheet (rfvhf.kicad_sch): BK4819 RX + 26MHz TCXO (2520) + PCM1808 ADC
- BK4819/PCM1808/TCXO_26M symbols added to project lib
- J3 airband pins: SCN/SCK/SDATA (GPIO29/30/47) + I2S2 MCLK/BCK/LRCK/DOUT (GPIO5/22/52/48)
- all passives 0603 (except RF ESD 0402); reuse existing BOM (only 3 new chips)
- BOM_V4.6_AIRBAND-zh_CN.md; PINMAP.md airband section
Other:
- added sheet RF_VHF (rfvhf.kicad_sch)
Changed lines of the file:
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@@
+		)
+	)
+	(sheet
+		(at 25.4 127)
+		(size 50.8 25.4)
+		(fields_autoplaced yes)
+		(stroke (width 0.1524) (type solid))
+		(fill (color 0 0 0 0.0000))
+		(property "Sheetname" "RF_VHF"
+			(at 25.4 126.2884 0)
+			(effects (font (size 1.27 1.27)) (justify left bottom))
+		)
+		(property "Sheetfile" "rfvhf.kicad_sch"
+			(at 25.4 152.9846 0)
+			(effects (font (size 1.27 1.27)) (justify left top))
+		)
+		(instances
+			(project "expansion-board-v4"
+				(path "/10000000-0000-4000-8000-000000000001" (page "8"))
+			)
 		)
 	)

Commit message: hardware(v4.7): 修正 C99 并刷新整套制造与装配文件
在用户修订的布局上将 C99 改为 100nF/0402，复用 C37/C52 的 C307331；同步原理图版本、BOM/CPL、装配图、安装助手及制造归档，更新下单入口和未决电气项。

验证：DRC 0 违规/0 未连通，存盘覆铜与包源一致性已核对；提交前版本包/安装助手20项，18通过、2跳过。元件契约中已记录的 C84 两条子断言失败按用户范围保留；Y4 供电和 U22 VREF 建议尚待闭环。内部工具、审计报告和采购过程文件按仓库规则仅留本地。
Other:
- title: Pilot Kit Expansion Board V1 - Root -> Pilot Kit Expansion Board V4.7 - Root
Changed lines of the file:
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@@
 	(paper "A3")
 	(title_block
-		(title "Pilot Kit Expansion Board V1 - Root")
+		(title "Pilot Kit Expansion Board V4.7 - Root")
 		(date "2026-08-01")
-		(rev "V1")
+		(rev "V4.7")
 		(company "Pilot Kit")
 		(comment 1 "Dual-band ADS-B (1090ES/978UAT) + IMU + BARO + GNSS")

Commit message: feat(v4.11): 固化扩展板并修正电池补偿
Other:
- title: Pilot Kit Expansion Board V4.7 - Root -> Pilot Kit Expansion Board V4.11 - Root
Changed lines of the file:
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@@
 	(paper "A3")
 	(title_block
-		(title "Pilot Kit Expansion Board V4.7 - Root")
+		(title "Pilot Kit Expansion Board V4.11 - Root")
 		(date "2026-08-01")
-		(rev "V4.7")
+		(rev "V4.11")
 		(company "Pilot Kit")
 		(comment 1 "Dual-band ADS-B (1090ES/978UAT) + IMU + BARO + GNSS")
