File: hardware/expansion-board-v4/kicad/interface.kicad_sch (KiCad schematic)
At the start: 1 part, among them J1 J3_HAT_2x20_SMD排针

Commit message: hardware(v4.6): airband BK4819 schematic + symbols + J3 wiring + BOM
- new RF_VHF sheet (rfvhf.kicad_sch): BK4819 RX + 26MHz TCXO (2520) + PCM1808 ADC
- BK4819/PCM1808/TCXO_26M symbols added to project lib
- J3 airband pins: SCN/SCK/SDATA (GPIO29/30/47) + I2S2 MCLK/BCK/LRCK/DOUT (GPIO5/22/52/48)
- all passives 0603 (except RF ESD 0402); reuse existing BOM (only 3 new chips)
- BOM_V4.6_AIRBAND-zh_CN.md; PINMAP.md airband section
Connections:
- net VHF_MCLK: now reaches J1.11 (Pin_11)
- net VHF_BCK: now reaches J1.17 (Pin_17)
- net VHF_SCN: now reaches J1.20 (Pin_20)
- net VHF_SCK: now reaches J1.22 (Pin_22)
- net VHF_SDATA: now reaches J1.37 (Pin_37)
- net VHF_LRCK: now reaches J1.38 (Pin_38)
- net VHF_DOUT: now reaches J1.39 (Pin_39)
- no-connect marks 20 -> 13
Changed lines of the file:
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@@
+		(effects (font (size 1.27 1.27)) (justify right))
+	)
+	(global_label "VHF_SCN"
+		(shape passive)
+		(at 109.22 88.9 0)
+		(effects (font (size 1.27 1.27)) (justify left))
+	)
+	(global_label "VHF_SCK"
+		(shape passive)
+		(at 109.22 91.44 0)
+		(effects (font (size 1.27 1.27)) (justify left))
+	)
+	(global_label "VHF_SDATA"
+		(shape passive)
+		(at 96.52 111.76 180)
+		(effects (font (size 1.27 1.27)) (justify right))
+	)
+	(global_label "VHF_MCLK"
+		(shape passive)
+		(at 96.52 78.74 180)
+		(effects (font (size 1.27 1.27)) (justify right))
+	)
+	(global_label "VHF_BCK"
+		(shape passive)
+		(at 96.52 86.36 180)
+		(effects (font (size 1.27 1.27)) (justify right))
+	)
+	(global_label "VHF_LRCK"
+		(shape passive)
+		(at 109.22 111.76 0)
+		(effects (font (size 1.27 1.27)) (justify left))
+	)
+	(global_label "VHF_DOUT"
+		(shape passive)
+		(at 96.52 114.3 180)
 		(effects (font (size 1.27 1.27)) (justify right))
 	)
@@
 	)
 	(no_connect
-		(at 96.52 78.74)
-	)
-	(no_connect
 		(at 109.22 78.74)
 	)
@@
 	)
 	(no_connect
-		(at 96.52 86.36)
-	)
-	(no_connect
 		(at 109.22 86.36)
 	)
 	(no_connect
-		(at 109.22 88.9)
-	)
-	(no_connect
 		(at 96.52 91.44)
-	)
-	(no_connect
-		(at 109.22 91.44)
 	)
 	(no_connect
@@
 		(at 109.22 101.6)
 	)
-	(no_connect
-		(at 96.52 111.76)
-	)
-	(no_connect
-		(at 109.22 111.76)
-	)
-	(no_connect
-		(at 96.52 114.3)
-	)
 	(embedded_fonts no)

Commit message: hardware(v4.7): 修正 C99 并刷新整套制造与装配文件
在用户修订的布局上将 C99 改为 100nF/0402，复用 C37/C52 的 C307331；同步原理图版本、BOM/CPL、装配图、安装助手及制造归档，更新下单入口和未决电气项。

验证：DRC 0 违规/0 未连通，存盘覆铜与包源一致性已核对；提交前版本包/安装助手20项，18通过、2跳过。元件契约中已记录的 C84 两条子断言失败按用户范围保留；Y4 供电和 U22 VREF 建议尚待闭环。内部工具、审计报告和采购过程文件按仓库规则仅留本地。
Other:
- title: Expansion Board V1 - Interface: J3 2x20 HAT socket -> Expansion Board V4.7 - Interface: J3 2x20 HAT socket
Changed lines of the file:
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@@
 	(paper "A3")
 	(title_block
-		(title "Expansion Board V1 - Interface: J3 2x20 HAT socket")
+		(title "Expansion Board V4.7 - Interface: J3 2x20 HAT socket")
 		(date "2026-08-01")
-		(rev "V1")
+		(rev "V4.7")
 		(company "Pilot Kit")
 	)

Commit message: feat(v4.11): 固化扩展板并修正电池补偿
Connections:
- net P4_GPIO4_SW3_SENSE: now reaches J1.14 (Pin_14)
- no-connect marks 13 -> 12
Other:
- title: Expansion Board V4.7 - Interface: J3 2x20 HAT socket -> Expansion Board V4.11 - Interface: J3 2x20 HAT socket
Changed lines of the file:
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@@
 	(paper "A3")
 	(title_block
-		(title "Expansion Board V4.7 - Interface: J3 2x20 HAT socket")
+		(title "Expansion Board V4.11 - Interface: J3 2x20 HAT socket")
 		(date "2026-08-01")
-		(rev "V4.7")
+		(rev "V4.11")
 		(company "Pilot Kit")
 	)
@@
 		(effects (font (size 1.27 1.27)) (justify left))
 	)
+	(global_label "P4_GPIO4_SW3_SENSE"
+		(shape passive)
+		(at 109.22 81.28 0)
+		(effects (font (size 1.27 1.27)) (justify left))
+	)
 	(global_label "GNSS_RXD"
 		(shape passive)
@@
 	)
 	(no_connect
-		(at 109.22 81.28)
-	)
-	(no_connect
