File: hardware/expansion-board-v4/kicad/mcu.kicad_sch (KiCad schematic)
At the start: 40 parts, among them J4 USB-C_16P, SW1 RESET短接焊盘, SW2 BOOTSEL短接焊盘, U8 RP2040, U9 W25Q128JVSIQ, Y1 12MHz CL=10pF ABM8-272-T3

Commit message: hardware(v4.7): 修正 C99 并刷新整套制造与装配文件
在用户修订的布局上将 C99 改为 100nF/0402，复用 C37/C52 的 C307331；同步原理图版本、BOM/CPL、装配图、安装助手及制造归档，更新下单入口和未决电气项。

验证：DRC 0 违规/0 未连通，存盘覆铜与包源一致性已核对；提交前版本包/安装助手20项，18通过、2跳过。元件契约中已记录的 C84 两条子断言失败按用户范围保留；Y4 供电和 U22 VREF 建议尚待闭环。内部工具、审计报告和采购过程文件按仓库规则仅留本地。
Other:
- title: Expansion Board V1 - MCU RP2040 + Flash + USB -> Expansion Board V4.7 - MCU RP2040 + Flash + USB
Changed lines of the file:
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@@
 	(paper "A3")
 	(title_block
-		(title "Expansion Board V1 - MCU RP2040 + Flash + USB")
+		(title "Expansion Board V4.7 - MCU RP2040 + Flash + USB")
 		(date "2026-08-01")
-		(rev "V1")
+		(rev "V4.7")
 		(company "Pilot Kit")
 	)

Commit message: hardware(v4.10): J11 改 2x10 测试焊盘阵列并入 airband；26MHz 探测点加隔离电阻 R66
J11 由 V4.9 的 2x8 贴片排针改成 2x10 裸焊盘阵列（自制封装
TestPad_2x10_P2.54mm：20 个 φ1.0mm 裸铜、2.54 网格、不贴任何件），
配 2x10p PCB 测试夹。中心上移 2.54mm，让新 pin5~20 精确落在原 pin1~16
的物理位置，16 根已布走线一根未动；但两列中心距从排针的 5.05mm 收到
探针的 2.54mm，20 个焊盘各内收 1.26mm，走线端点随之跟进。

两处会让人照旧图读错板的改动：
- 脚号整体后移 4 位，且跳线帽消失、三对短接改用镊子/锡桥
  （复位 1-2→5-6、BOOTSEL 3-4→7-8、自检回环 15-16→19-20）。
- 焊盘定 φ1.0 而不是 φ1.2：两列之间要并排走 4 根 0.15mm 线，
  按 0.15 间距需 1.35mm 净宽，φ1.2 只剩 1.34mm，差 0.01mm 塞不下。

新增 airband 四脚（VHF_TCXO_TP / VHF_AUDIO / VHF_SCK / VHF_SDATA），
沿板子下缘布通，在 1090 接收前端所在的 y 50.5~58 带内铜长 0.0mm。
26MHz 参考经 R66（0Ω 0603，**默认不贴**）隔离：那根分支 119.9mm 走 In2，
直连会给 TG-5006CG 加约 17pF，而手册 Output load 是 10kΩ // 10pF、
fo-Load 条件栏写死 ±10%。频率不是主要风险，幅度才是——0.8Vpp Min 是在
10pF 下保证的，27pF 在 26MHz 只剩 227Ω，而 BK4819 的 XI 是并联谐振晶体口、
手册没给外部注入门限，参考起不来就是 airband 整条收不了。
R66 必须在 TCXO 端；放 J11 端那 120mm 仍挂在振荡节点上，等于白做。
不贴时振荡节点残留 11.0mm + 2 过孔 ≈ 1.8pF。

丝印：B 面 20 格图例 + J11 旁竖排行号（偶数脚 2~20，与焊盘行逐行对齐，
离本体 1.0mm）。图例与 J11 位号的最终位置由维护者手工定稿后固化，
独立的 "J11" 板级文字因与位号重复已删除。

顺带修掉四处会静默出错的地方：
- gen_j11_silk 的障碍模型错了三次：B.SilkS 层名比对恒假（避让从未生效）、
  改宽后把 F 面丝印和 F 面贴片焊盘也当成 B 面丝印的障碍（误判"放不下"）。
  已按"只算 B 面"收敛，并加防覆盖闸：板上已有整套图例时拒绝重排。
- SHORT 漏缩写会让单元格回退成完整网名，那串既不匹配 drop 的正则、
  又撑爆表格布局，在板上越积越多；已加覆盖断言。
- R66 的「默认不贴」要在五份名单里登记，gen_master_bom 的护栏当场抓到漏项。
- 合同补上行号列与图例的位置断言，不只查文字存在。

验证：DRC 0 违例 / 0 未连通 / 丝印 0 违例；文档坐标 438 处 0 处对不上；
硬件合同 73 passed / 8 skipped。check_gerber 的 ⑤ 项与历史包逐字相同，
是本板恒报的 SW3 机械固定脚，非本轮引入。

发布包：V4.8 移出 release/（留档 build/v48-superseded/），
V4.9 按已下单存入 release/archive/20260915-V4.9-ordered/，
当前可下单为 V4.10-20260921。
Parts:
- removed SW1: RESET短接焊盘, Jumper:SolderJumper-2_P1.3mm_Open_Pad1.0x1.5mm, symbol Jumper:SolderJumper_2_Open
- removed SW2: BOOTSEL短接焊盘, Jumper:SolderJumper-2_P1.3mm_Open_Pad1.0x1.5mm, symbol Jumper:SolderJumper_2_Open
- removed TP1, TP2, TP3, TP4, TP5, TP6, TP7: TestPoint, TestPoint:TestPoint_Pad_1.0x1.0mm, symbol Connector:TestPoint
- added J11: 调试焊盘阵列 2x10, expansion-board-v4:TestPad_2x10_P2.54mm, symbol Connector_Generic:Conn_02x10_Odd_Even
Connections:
- net DEMOD0: now also J11.14 (Pin_14)
- net DEMOD1: now also J11.16 (Pin_16)
- net DEMOD2: now also J11.18 (Pin_18)
- net DEMOD3: now also J11.17 (Pin_17)
- net GND: now also J11.15 (Pin_15), J11.5 (Pin_5), J11.7 (Pin_7)
- net PULSES: now also J11.20 (Pin_20)
- net QSPI_SS: now also J11.8 (Pin_8)
- net RECOVERED_CLK: now also J11.19 (Pin_19)
- net RP_RUN: now also J11.6 (Pin_6)
- net SUBG_RESET: now also J11.13 (Pin_13)
- net SUBG_TCKC: now also J11.11 (Pin_11)
- net SUBG_TMSC: now also J11.9 (Pin_9)
- net SWCLK: now also J11.10 (Pin_10)
- net SWDIO: now also J11.12 (Pin_12)
- new net VHF_AUDIO: J11.2 (Pin_2)
- new net VHF_SCK: J11.3 (Pin_3)
- new net VHF_SDATA: J11.4 (Pin_4)
- new net VHF_TCXO_TP: J11.1 (Pin_1)
Other:
- title: Expansion Board V4.7 - MCU RP2040 + Flash + USB -> Expansion Board V4.10 - MCU RP2040 + Flash + USB

Commit message: feat(v4.11): 固化扩展板并修正电池补偿
Other:
- title: Expansion Board V4.10 - MCU RP2040 + Flash + USB -> Expansion Board V4.11 - MCU RP2040 + Flash + USB
Changed lines of the file:
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@@
 	(paper "A3")
 	(title_block
-		(title "Expansion Board V4.10 - MCU RP2040 + Flash + USB")
+		(title "Expansion Board V4.11 - MCU RP2040 + Flash + USB")
 		(date "2026-08-01")
-		(rev "V4.10")
+		(rev "V4.11")
 		(company "Pilot Kit")
 	)
