File: hardware/expansion-board-v4/kicad/rf1090.kicad_sch (KiCad schematic)
At the start: 56 parts, among them J6 U.FL_1090_EXT(经尾线转SMA), J7 U.FL_IFA_TEST(π后调试口), Q3 AO3401A, U11 QPL9547TR7, U12 BGA2817, U14 AD8313ARMZ, U15 TLV3501(TOKMAS), U16 XA17-G4K

Commit message: hardware(v4.7): 修正 C99 并刷新整套制造与装配文件
在用户修订的布局上将 C99 改为 100nF/0402，复用 C37/C52 的 C307331；同步原理图版本、BOM/CPL、装配图、安装助手及制造归档，更新下单入口和未决电气项。

验证：DRC 0 违规/0 未连通，存盘覆铜与包源一致性已核对；提交前版本包/安装助手20项，18通过、2跳过。元件契约中已记录的 C84 两条子断言失败按用户范围保留；Y4 供电和 U22 VREF 建议尚待闭环。内部工具、审计报告和采购过程文件按仓库规则仅留本地。
Other:
- title: Expansion Board V1 - 1090MHz: antenna switch + RX chain -> Expansion Board V4.7 - 1090MHz: antenna switch + RX chain
Changed lines of the file:
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@@
 	(paper "A3")
 	(title_block
-		(title "Expansion Board V1 - 1090MHz: antenna switch + RX chain")
+		(title "Expansion Board V4.7 - 1090MHz: antenna switch + RX chain")
 		(date "2026-08-01")
-		(rev "V1")
+		(rev "V4.7")
 		(company "Pilot Kit")
 	)

Commit message: feat(v4.11): 固化扩展板并修正电池补偿
Other:
- title: Expansion Board V4.7 - 1090MHz: antenna switch + RX chain -> Expansion Board V4.11 - 1090MHz: antenna switch + RX chain
Changed lines of the file:
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@@
 	(paper "A3")
 	(title_block
-		(title "Expansion Board V4.7 - 1090MHz: antenna switch + RX chain")
+		(title "Expansion Board V4.11 - 1090MHz: antenna switch + RX chain")
 		(date "2026-08-01")
-		(rev "V4.7")
+		(rev "V4.11")
 		(company "Pilot Kit")
 	)
